Commit message: Update wheels.xacro

File: mybot_description/urdf/wheels.xacro (robot description, xacro)
@@ -38,4 +38,7 @@
       <parent link='base_link'/>
     </joint>
+    <gazebo reference = '${prefix}_wheel'>
+      <material>Gazebo/Yellow</material>
+    </gazebo>
   </xacro:macro>
   <xacro:wheel prefix='left' reflect='1'/>
